File: Schematics/start.sch (EAGLE design)
At the start: 6 parts, among them U2 TINY85-20-DIP

Commit message: Initial commit of start sensor schematic.
Parts:
- removed JP2: (no value), SparkFun-Connectors:M081X08
- added JP1: M10", SparkFun-Connectors:M10"
- renumbered LED2 to LED1, R10 to R3, R6 to R1, R9 to R2, U2 to U1
Connections:
- net 5V: now also JP1.6, JP1.7; no longer JP2.2, JP2.5
- net GND: now also JP1.10, JP1.4, JP1.5, JP1.8; no longer JP2.3, JP2.4, JP2.6, JP2.8
- net SIGIN: now also JP1.9; no longer JP2.7
- net TX: now also JP1.1; no longer JP2.1
Other:
- note added: "Connections 1,2,3,4 - PROP PLUG (Serial to USB) 5,6 - Power Input 7,8,9,10 - Power and Signal to other sensor"
- note removed: "Pin Definitions 1. Serial data out 2. 5V in 5. 5V to finish sensor 7. Data wire from finish sensor NOTE: Pins 5,6,7,8 are connected to finish sensor via telephone cord."
